File: pcb/keebykeeb.kicad_sch (KiCad schematic)
At the start: 182 parts, among them J1 USB_C_Receptacle, J2 USB_C_Receptacle, J3 USB_C_Receptacle, J4 USB_C_Receptacle, J5 USB3_A, J6 USB3_A, J7 USB_C_Receptacle, J8 USB_C_Receptacle, SW1 SW_Push, SW10 SW_Push, SW11 SW_Push, SW12 SW_Push, SW13 SW_Push, SW14 SW_Push, SW15 SW_Push, SW16 SW_Push, SW17 SW_Push, SW18 SW_Push, SW19 SW_Push, SW2 SW_Push, SW20 SW_Push, SW21 SW_Push, SW22 SW_Push, SW23 SW_Push, SW24 SW_Push, SW25 SW_Push, SW26 SW_Push, SW27 SW_Push, SW28 SW_Push, SW29 SW_Push, SW3 SW_Push, SW30 SW_Push, SW31 SW_Push, SW32 SW_Push, SW33 SW_Push, SW34 SW_Push, SW35 SW_Push, SW36 SW_Push, SW37 SW_Push, SW38 SW_Push, SW39 SW_Push, SW4 SW_Push, SW40 SW_Push, SW41 SW_Push, SW42 SW_Push, SW43 SW_Push, SW44 SW_Push, SW45 SW_Push, SW46 SW_Push, SW47 SW_Push, SW48 SW_Push, SW49 SW_Push, SW5 SW_Push, SW50 SW_Push, SW51 SW_Push, SW52 SW_Push, SW53 SW_Push, SW54 SW_Push, SW55 SW_Push, SW56 SW_Push, SW57 SW_Push, SW58 SW_Push, SW59 SW_Push, SW6 SW_Push, SW60 SW_Push, SW61 SW_Push, SW62 SW_Push, SW63 SW_Push, SW64 SW_Push, SW65 SW_Push, SW66 SW_Push, SW67 SW_Push, SW68 SW_Push, SW69 SW_Push, SW7 SW_Push, SW70 SW_Push, SW71 SW_Push, SW72 SW_Push, SW73 SW_Push, SW74 SW_Push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

Commit message: omg i gotta do ESD protection now
Parts:
- removed J1, J3, J4: USB_C_Receptacle, symbol Connector:USB_C_Receptacle
- removed J6: USB3_A, symbol Connector:USB3_A
- removed R10, R11, R9: 0, symbol Device:R
- removed R2, R4, R5, R6, R7, R8: 200K, symbol Device:R
- removed R3: 900K, symbol Device:R
- removed U5: HD3SS3220IRNHR, RNH0030A, symbol HD3SS3220:HD3SS3220IRNHR
- added C10, C11, C12, C9: 100nF, symbol Device:C_Small
- added C4, C5, C8: 0.1µF, symbol Device:C_Small
- added D77: SMAJ5.0A, Diode_SMD:D_SMA, symbol Diode:SMAJ5.0A
- added FB1: 220@100MHz, symbol Device:FerriteBead_Small
- added J10, J9: USB_C_Receptacle, symbol Connector:USB_C_Receptacle
- added J11: USB3_A, symbol Connector:USB3_A
- added R26, R37, R48: 0, symbol Device:R
- added R27, R39, R49: 100K, symbol Device:R
- added R29: 909K, symbol Device:R
- added R30, R31, R32, R34: 200K, symbol Device:R
- added R33: 4.7k, symbol Device:R
- added R46: 90.9K, symbol Device:R
- added R47: 10K, symbol Device:R
- added U10, U15, U9: TPS2552DDBVR, DBV0006A_TEX, symbol TPS2552:TPS2552DDBVR
- added U11, U14: HD3SS3220IRNHR, RNH0030A, symbol HD3SS3220:HD3SS3220IRNHR
Connections:
- net +3V3: now also R30.1
- net +5V: now also J7.A4 (VBUS), J7.A9 (VBUS), J7.B4 (VBUS), J7.B9 (VBUS), C4.2, C5.2, C8.2, D77.1 (A1), R27.2, R31.1, R32.1, R33.1, R34.1, R39.2, R46.1, R49.2, U10.1 (IN), U15.1 (IN), U9.1 (IN)
- net GND: now also J7.A1 (GND), J7.A12 (GND), J7.B1 (GND), J7.B12 (GND), J7.SH (SHIELD), C4.1, C5.1, C8.1, D77.2 (A2), J10.A1 (GND), J10.A12 (GND), J10.B1 (GND), J10.B12 (GND), J10.SH (SHIELD), J9.A1 (GND), J9.A12 (GND), J9.B1 (GND), J9.B12 (GND), J9.SH (SHIELD), R26.2, R37.2, R47.2, R48.2, U10.2 (GND), U11.12 (EN_MUX_N), U11.13 (GND), U11.28 (GND), U11.29 (EN_CC_N), U11.31 (PAD), U15.2 (GND), U9.2 (GND)
- net HPC_DP: now reaches U1.17 (USB_DP_DN3)
- net HPC_DP: now also J10.A6 (D+), J10.B6 (D+)
- net HPC_DM: now reaches U1.18 (USB_DM_DN3)
- net HPC_DM: now also J10.A7 (D-), J10.B7 (D-)
- net HPC_TXP: now reaches U1.19 (USB_SSTXP_DN3)
- net HPC_TXP: now also U11.6 (TXP)
- net HPC_TXM: now reaches U1.20 (USB_SSTXM_DN3)
- net HPC_TXM: now also U11.7 (TXN)
- net HPC_RXP: now reaches U1.22 (USB_SSRXP_DN3)
- net HPC_RXP: now also U11.9 (RXP)
- net HPC_RXM: now reaches U1.23 (USB_SSRXM_DN3)
- net HPC_RXM: now also U11.10 (RXN)
- net HPA_DP: now reaches U1.24 (USB_DP_DN4)
- net HPA_DM: now reaches U1.25 (USB_DM_DN4)
- net HPA_TXP: now reaches U1.26 (USB_SSTXP_DN4)
- net HPA_TXM: now reaches U1.27 (USB_SSTXM_DN4)
- net HPA_RXP: now reaches U1.29 (USB_SSRXP_DN4)
- net HPA_RXM: now reaches U1.30 (USB_SSRXM_DN4)
- net HPA_EN: now reaches U1.32 (PWRCTL4_BATEN4)
- net HPC_EN: now reaches U1.33 (PWRCTL3_BATEN3)
- net HPC_EN: now also U10.3 (EN)
- net EXT_EN: now reaches U1.35 (PWRCTL2_BATEN2)
- net EXT_EN: now also U15.3 (EN), U9.3 (EN)
- net HPA_FAULT: now reaches U1.43 (OVERCUR4_N)
- net HPC_FAULT: now reaches U1.44 (OVERCUR3_N)
- net HPC_FAULT: now also R39.1, U10.4 (*FAULT)
- net EXT_FAULT: now reaches U1.47 (OVERCUR2_N)
- net EXT_FAULT: now also R27.1, R49.1, U15.4 (*FAULT), U9.4 (*FAULT)
- net at U1.48 (USB_VBUS): now also R46.2, R47.1
- net LPC_DM: now reaches U2.10 (USB_DM_DN2)
- net LPC_DM: now also J9.A7 (D-), J9.B7 (D-)
- net LPC_TXP: now reaches U2.11 (USB_SSTXP_DN2)
- net LPC_TXM: now reaches U2.12 (USB_SSTXM_DN2)
- net LPC_RXP: now reaches U2.14 (USB_SSRXP_DN2)
- net LPC_RXM: now reaches U2.15 (USB_SSRXM_DN2)
- net LPCADP: now reaches U2.17 (USB_DP_DN3)
- net LPA_DM: now reaches U2.18 (USB_DM_DN3)
- net LPA_DM: now also J11.2 (D-)
- net LPA_TXP: now reaches U2.19 (USB_SSTXP_DN3)
- net LPA_TXP: now also J11.9 (SSTX+)
- net LPA_TXM: now reaches U2.20 (USB_SSTXM_DN3)
- net LPA_TXM: now also J11.8 (SSTX-)
- net LPA_RXP: now reaches U2.22 (USB_SSRXP_DN3)
- net LPA_RXP: now also J11.6 (SSRX+)
- net LPA_RXM: now reaches U2.23 (USB_SSRXM_DN3)
- net LPA_RXM: now also J11.5 (SSRX-)
- net LPA_EN: now reaches U2.33 (PWRCTL3_BATEN3)
- net LPC_EN: now reaches U2.35 (PWRCTL2_BATEN2)
- net KB_EN: now reaches U2.36 (PWRCTL1_BATEN1)
- net LPA_FAULT: now reaches U2.44 (OVERCUR3_N)
- net KB_FAULT: now reaches U2.46 (OVERCUR1_N)
- net LPC_FAULT: now reaches U2.47 (OVERCUR2_N)
- net LPC_DP: now reaches U2.9 (USB_DP_DN2)
- net LPC_DP: now also J9.A6 (D+), J9.B6 (D+)
- net at J7.A10 (RX2-): now also U14.18 (RX2N)
- net at J7.A11 (RX2+): now also U14.19 (RX2P)
- net at J7.A2 (TX1+): now also U14.17 (TX1P)
- net at J7.A3 (TX1-): now also U14.16 (TX1N)
- net at J7.A5 (CC1): now also U14.2 (CC1)
- net at J7.B10 (RX1-): now also U14.14 (RX1N)
- net at J7.B11 (RX1+): now also U14.15 (RX1P)
- net at J7.B2 (TX2+): now also U14.21 (TX2P)
- net at J7.B3 (TX2-): now also U14.20 (TX2N)
- net at J7.B5 (CC2): now also U14.1 (CC2)
- net at J2.A4 (VBUS), J2.A9 (VBUS), J2.B4 (VBUS)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: now also U9.6 (OUT)
- new net: R34.2, U11.24 (VCONN_FAULT_N)
- new net: R48.1, U15.5 (ILIM)
- new net: R37.1, U10.5 (ILIM)
- new net: R31.2, U11.23 (INT_OUT3_N)
- new net: C9.1, J10.A3 (TX1-)
- new net: C9.2, U11.16 (TX1N)
- new net: C10.1, J10.A2 (TX1+)
- new net: C10.2, U11.17 (TX1P)
- new net: R26.1, U9.5 (ILIM)
- new net: J9.A4 (VBUS), J9.A9 (VBUS), J9.B4 (VBUS), J9.B9 (VBUS)
- new net: J10.A10 (RX2-), U11.18 (RX2N)
- new net: J10.A11 (RX2+), U11.19 (RX2P)
- new net: J10.A5 (CC1), U11.2 (CC1)
- new net: J10.B10 (RX1-), U11.14 (RX1N)
- new net: J10.B11 (RX1+), U11.15 (RX1P)
- new net: C11.1, J10.B2 (TX2+)
- new net: C12.1, J10.B3 (TX2-)
- new net: J10.B5 (CC2), U11.1 (CC2)
- new net: R32.2, U11.27 (ID)
- new net: R33.2, U11.4 (PORT)
- new net: C11.2, U11.21 (TX2P)
- new net: R29.2, U11.5 (VBUS_DET)
- new net: R30.2, U11.11 (DIR)
- new net: C12.2, U11.20 (TX2N)
- new net HPC_VBUS: J10.A4 (VBUS), J10.A9 (VBUS), J10.B4 (VBUS), J10.B9 (VBUS), R29.1, U10.6 (OUT)
- new net LPA_DP: J11.3 (D+)
- no-connect marks 26 -> 42
Other:
- note added: "LOW POWER PORTS"
- note added: "sets current limit ()"
- moved on the sheet: C1, J2, J5, J8, R1, U3, U4
